File: bldc_motor_controller.kicad_pcb (KiCad board)
At the start: 2 copper layers, 50 x 50 mm, 43 parts, among them K1 CONN_3, P5 CONN_2, P6 CONN_3, P8 CONN_9, U1 TM4C1232XXPM, U2 LP2985LV, U4 L6234

Commit message: Fix proper wide tracks for m_sense, which carries all the motor currents.
Parts:
- moved R9 16.9 mm to (44.8, 79.9), turned to 0 degrees
- moved R10 13.1 mm to (44.6, 60.6), turned to 0 degrees
- moved C19 2.55 mm to (41.3, 58.0), turned to 135 degrees
- moved C18 1.70 mm to (46.9, 57.4)
Routing:
- net GND: track 143.3 -> 115.1 mm, vias 64 -> 62
- net /vboot: track 9.27 -> 11.6 mm
- net /m_en2: track 66.7 -> 68.5 mm
- net /m_in1: track 52.1 -> 50.3 mm
- net /vcp: track 3.74 -> 5.44 mm
- net /m_in2: track 71.2 -> 72.7 mm
- net /m_sense2_raw: track 21.3 -> 20.4 mm
